File: wang600-docs/kicad/5929-core-drive/5929-core-drive.kicad_sch (KiCad schematic)
At the start: 33 parts, among them Q25 2N3640, Q26 GT544, Q27 GT545, Q60 GT545, Q61 GT544, U1 SN7525N, U17 7400, U6 7400, U7 7400

Commit message: yet more schematic cleanup
Other:
- title: (none) -> Wang 700 Magentic Core Memory
Changed lines of the file:
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@@
 (kicad_sch (version 20211123) (generator eeschema)
   (paper "A4")
+  (title_block
+    (title "Wang 700 Magentic Core Memory")
+    (date "2024-04-15")
+  )
   (junction (at 107.315 26.67) (diameter 0) (color 0 0 0 0)
   )
@@
   )
   (polyline (pts (xy 76.2 117.475) (xy 76.2 120.65))
-    (stroke (width 0) (type solid) (color 0 0 194 1))
+    (stroke (width 0) (type solid) (color 0 0 0 1))
   )
   (wire (pts (xy 120.65 26.67) (xy 107.315 26.67))
@@
   )
   (polyline (pts (xy 44.45 120.65) (xy 54.61 117.475))
-    (stroke (width 0) (type solid) (color 0 0 194 1))
+    (stroke (width 0) (type solid) (color 0 0 0 1))
   )
   (wire (pts (xy 240.665 28.575) (xy 250.825 28.575))
@@
   )
   (polyline (pts (xy 25.4 127) (xy 63.5 127))
-    (stroke (width 0) (type solid) (color 0 0 194 1))
+    (stroke (width 0) (type solid) (color 0 0 0 1))
   )
   (wire (pts (xy 107.315 26.67) (xy 94.615 26.67))
@@
   )
   (polyline (pts (xy 26.035 111.125) (xy 44.45 111.125))
-    (stroke (width 0) (type solid) (color 0 0 194 1))
+    (stroke (width 0) (type solid) (color 0 0 0 1))
   )
   (wire (pts (xy 153.67 151.13) (xy 168.91 151.13))
@@
   )
   (polyline (pts (xy 66.04 127) (xy 82.55 127))
-    (stroke (width 0) (type solid) (color 0 0 194 1))
+    (stroke (width 0) (type solid) (color 0 0 0 1))
   )
   (bus (pts (xy 209.55 89.535) (xy 209.55 114.3))
@@
   )
   (polyline (pts (xy 76.2 120.65) (xy 82.55 120.65))
-    (stroke (width 0) (type solid) (color 0 0 194 1))
+    (stroke (width 0) (type solid) (color 0 0 0 1))
   )
   (bus (pts (xy 171.45 82.55) (xy 171.45 89.535))
@@
   )
   (polyline (pts (xy 25.4 120.65) (xy 44.45 120.65))
-    (stroke (width 0) (type solid) (color 0 0 194 1))
+    (stroke (width 0) (type solid) (color 0 0 0 1))
   )
   (wire (pts (xy 72.39 26.67) (xy 81.915 26.67))
@@
   )
   (polyline (pts (xy 38.1 133.35) (xy 44.45 133.35))
-    (stroke (width 0) (type solid) (color 0 0 194 1))
+    (stroke (width 0) (type solid) (color 0 0 0 1))
   )
   (polyline (pts (xy 278.765 19.05) (xy 278.765 56.515))
@@
   )
   (polyline (pts (xy 38.1 130.175) (xy 38.1 133.35))
-    (stroke (width 0) (type solid) (color 0 0 194 1))
+    (stroke (width 0) (type solid) (color 0 0 0 1))
   )
   (wire (pts (xy 43.815 26.67) (xy 55.245 26.67))
@@
   )
   (polyline (pts (xy 63.5 123.19) (xy 66.04 127))
-    (stroke (width 0) (type solid) (color 0 0 194 1))
+    (stroke (width 0) (type solid) (color 0 0 0 1))
   )
   (bus (pts (xy 209.55 82.55) (xy 209.55 89.535))
@@
   )
   (polyline (pts (xy 44.45 133.35) (xy 44.45 130.175))
-    (stroke (width 0) (type solid) (color 0 0 194 1))
+    (stroke (width 0) (type solid) (color 0 0 0 1))
   )
   (polyline (pts (xy 165.1 107.315) (xy 165.1 73.025))
@@
   )
   (polyline (pts (xy 76.2 114.3) (xy 76.2 110.49))
-    (stroke (width 0) (type solid) (color 0 0 194 1))
+    (stroke (width 0) (type solid) (color 0 0 0 1))
   )
   (wire (pts (xy 173.99 62.865) (xy 184.15 62.865))
@@
   )
   (polyline (pts (xy 76.2 110.49) (xy 82.55 110.49))
-    (stroke (width 0) (type solid) (color 0 0 194 1))
+    (stroke (width 0) (type solid) (color 0 0 0 1))
   )
   (wire (pts (xy 140.97 157.48) (xy 146.05 157.48))
@@
   )
   (polyline (pts (xy 25.4 139.7) (xy 63.5 139.7))
-    (stroke (width 0) (type solid) (color 0 0 194 1))
+    (stroke (width 0) (type solid) (color 0 0 0 1))
   )
   (polyline (pts (xy 63.5 135.89) (xy 69.85 135.89))
-    (stroke (width 0) (type solid) (color 0 0 194 1))
+    (stroke (width 0) (type solid) (color 0 0 0 1))
   )
   (wire (pts (xy 81.915 71.755) (xy 81.915 67.31))
@@
   )
   (polyline (pts (xy 44.45 130.175) (xy 82.55 130.175))
-    (stroke (width 0) (type solid) (color 0 0 194 1))
+    (stroke (width 0) (type solid) (color 0 0 0 1))
   )
   (polyline (pts (xy 257.175 104.775) (xy 257.175 71.12))
@@
   )
   (polyline (pts (xy 69.85 135.89) (xy 69.85 139.7))
-    (stroke (width 0) (type solid) (color 0 0 194 1))
+    (stroke (width 0) (type solid) (color 0 0 0 1))
   )
   (wire (pts (xy 192.405 107.315) (xy 193.04 107.315))
@@
   )
   (polyline (pts (xy 44.45 114.3) (xy 76.2 114.3))
-    (stroke (width 0) (type solid) (color 0 0 194 1))
+    (stroke (width 0) (type solid) (color 0 0 0 1))
   )
   (wire (pts (xy 107.315 71.755) (xy 94.615 71.755))
@@
   )
   (polyline (pts (xy 25.4 130.175) (xy 38.1 130.175))
-    (stroke (width 0) (type solid) (color 0 0 194 1))
+    (stroke (width 0) (type solid) (color 0 0 0 1))
   )
   (wire (pts (xy 117.475 90.805) (xy 113.03 90.805))
@@
   )
   (polyline (pts (xy 44.45 111.125) (xy 44.45 114.3))
-    (stroke (width 0) (type solid) (color 0 0 194 1))
+    (stroke (width 0) (type solid) (color 0 0 0 1))
   )
   (polyline (pts (xy 69.85 139.7) (xy 82.55 139.7))
-    (stroke (width 0) (type solid) (color 0 0 194 1))
+    (stroke (width 0) (type solid) (color 0 0 0 1))
   )
   (wire (pts (xy 94.615 71.755) (xy 81.915 71.755))
@@
   )
   (polyline (pts (xy 63.5 127) (xy 63.5 123.19))
-    (stroke (width 0) (type solid) (color 0 0 194 1))
+    (stroke (width 0) (type solid) (color 0 0 0 1))
   )
   (bus (pts (xy 202.565 102.235) (xy 202.565 143.51))
@@
   )
   (polyline (pts (xy 54.61 117.475) (xy 76.2 117.475))
-    (stroke (width 0) (type solid) (color 0 0 194 1))
+    (stroke (width 0) (type solid) (color 0 0 0 1))
   )
   (polyline (pts (xy 63.5 139.7) (xy 63.5 135.89))
-    (stroke (width 0) (type solid) (color 0 0 194 1))
+    (stroke (width 0) (type solid) (color 0 0 0 1))
   )
   (wire (pts (xy 138.43 26.67) (xy 120.65 26.67))

Commit message: still more schematic cleanup
Parts:
- D? (x4): value D -> Si
- gave numbers to parts that had none: 8
Other:
- note added: "Diodes placed remote for sensing PCB 6038 operating temperature"
- note added: "measure to Vdd"
