File: wang600-docs/kicad/5938-wire-weave-rom/5938-wire-weave-rom.kicad_sch (KiCad schematic)
At the start: 34 parts, among them Q32 GT544, Q33 GT544, Q34 2N4038, Q35 2N3014, U11 7401, U38 74LS04

Commit message: yet more schematic cleanup
Parts:
- removed TP1: TestPoint, symbol Connector:TestPoint
Connections:
- net LBIT is gone; now on net BIT: U?.3, U?.4
- net BIT: no longer Q35.2 (C), R?.2, U?.1
- net energize: now reaches C4.2, D1.1 (K), Q33.3 (B), Q34.1 (C), R100.1
- new net /BIT: Q35.2 (C), R?.2, U?.1
Other:
- note added: "/BIT"
- note added: "energize"
- note removed: "BIT"
- note removed: "TP1"
- title: (none) -> Wang 700 Wire-Weave ROM
Changed lines of the file:
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@@
 (kicad_sch (version 20211123) (generator eeschema)
   (paper "A4")
-  (junction (at 130.175 55.245) (diameter 0) (color 0 0 0 0)
+  (title_block
+    (title "Wang 700 Wire-Weave ROM")
+    (date "2024-04-15")
   )
   (junction (at 217.17 142.24) (diameter 0) (color 0 0 0 0)
@@
   (junction (at 100.33 23.495) (diameter 0) (color 0 0 0 0)
   )
+  (junction (at 224.79 142.24) (diameter 0) (color 0 0 0 0)
+  )
   (junction (at 196.85 154.94) (diameter 0) (color 0 0 0 0)
   )
@@
   )
   (junction (at 112.395 181.61) (diameter 0) (color 0 0 0 0)
+  )
+  (junction (at 125.095 55.245) (diameter 0) (color 0 0 0 0)
   )
   (junction (at 189.23 154.94) (diameter 0) (color 0 0 0 0)
@@
     (stroke (width 0) (type default) (color 0 0 0 0))
   )
-  (wire (pts (xy 217.17 142.24) (xy 222.885 142.24))
+  (wire (pts (xy 217.17 142.24) (xy 224.79 142.24))
     (stroke (width 0) (type default) (color 0 0 0 0))
   )
@@
     (stroke (width 0) (type default) (color 0 0 0 0))
   )
-  (polyline (pts (xy 235.585 121.285) (xy 235.585 163.195))
+  (wire (pts (xy 224.79 142.24) (xy 229.235 142.24))
+    (stroke (width 0) (type default) (color 0 0 0 0))
+  )
+  (polyline (pts (xy 236.855 121.285) (xy 236.855 163.195))
     (stroke (width 0) (type default) (color 0 0 0 0))
   )
@@
     (stroke (width 0) (type default) (color 0 0 0 0))
   )
+  (wire (pts (xy 127 49.53) (xy 125.095 49.53))
+    (stroke (width 0) (type default) (color 0 0 0 0))
+  )
   (bus (pts (xy 189.865 83.82) (xy 189.865 89.535))
     (stroke (width 0) (type default) (color 0 0 0 0))
@@
     (stroke (width 0) (type default) (color 0 0 0 0))
   )
-  (polyline (pts (xy 235.585 163.195) (xy 278.13 163.195))
+  (polyline (pts (xy 236.855 163.195) (xy 278.13 163.195))
     (stroke (width 0) (type default) (color 0 0 0 0))
   )
@@
     (stroke (width 0) (type solid) (color 0 0 0 1))
   )
+  (wire (pts (xy 125.095 55.245) (xy 138.43 55.245))
+    (stroke (width 0) (type default) (color 0 0 0 0))
+  )
   (polyline (pts (xy 47.625 129.54) (xy 47.625 133.35))
     (stroke (width 0) (type solid) (color 0 0 0 1))
@@
     (stroke (width 0) (type solid) (color 0 0 0 1))
   )
-  (wire (pts (xy 242.57 131.445) (xy 246.38 131.445))
+  (wire (pts (xy 224.79 131.445) (xy 246.38 131.445))
     (stroke (width 0) (type default) (color 0 0 0 0))
   )
@@
     (stroke (width 0) (type solid) (color 0 0 0 1))
   )
-  (wire (pts (xy 130.175 55.245) (xy 138.43 55.245))
-    (stroke (width 0) (type default) (color 0 0 0 0))
-  )
-  (polyline (pts (xy 235.585 121.285) (xy 278.13 121.285))
+  (polyline (pts (xy 236.855 121.285) (xy 278.13 121.285))
     (stroke (width 0) (type default) (color 0 0 0 0))
   )
@@
     (stroke (width 0) (type default) (color 0 0 0 0))
   )
-  (polyline (pts (xy 229.235 163.195) (xy 170.815 163.195))
+  (polyline (pts (xy 227.965 163.195) (xy 170.815 163.195))
     (stroke (width 0) (type default) (color 0 0 0 0))
   )
@@
     (stroke (width 0) (type default) (color 204 102 0 1))
   )
-  (polyline (pts (xy 229.235 121.285) (xy 229.235 163.195))
+  (polyline (pts (xy 227.965 121.285) (xy 227.965 163.195))
     (stroke (width 0) (type default) (color 0 0 0 0))
   )
@@
     (stroke (width 0) (type default) (color 0 0 0 0))
   )
-  (polyline (pts (xy 183.515 121.285) (xy 229.235 121.285))
+  (polyline (pts (xy 183.515 121.285) (xy 227.965 121.285))
     (stroke (width 0) (type default) (color 0 0 0 0))
   )
@@
     (stroke (width 0) (type default) (color 0 0 0 0))
   )
+  (wire (pts (xy 125.095 49.53) (xy 125.095 55.245))
+    (stroke (width 0) (type default) (color 0 0 0 0))
+  )
   (wire (pts (xy 199.39 86.995) (xy 202.565 86.995))
     (stroke (width 0) (type default) (color 0 0 0 0))
@@
     (stroke (width 0) (type default) (color 0 0 0 0))
   )
+  (wire (pts (xy 224.79 131.445) (xy 224.79 142.24))
+    (stroke (width 0) (type default) (color 0 0 0 0))
+  )
   (wire (pts (xy 67.31 51.435) (xy 67.31 46.99))
     (stroke (width 0) (type default) (color 0 0 0 0))
@@
     (stroke (width 0) (type default) (color 0 0 0 0))
   )
-  (wire (pts (xy 113.03 55.245) (xy 130.175 55.245))
+  (wire (pts (xy 113.03 55.245) (xy 125.095 55.245))
     (stroke (width 0) (type default) (color 0 0 0 0))
   )
@@
     (effects (font (size 1.27 1.27)) (justify right bottom))
   )
-  (text "BIT" (at 31.75 139.065 180)
+  (text "/BIT" (at 31.75 139.065 180)
     (effects (font (size 1.27 1.27)) (justify right bottom))
   )
@@
     (effects (font (size 1.27 1.27)) (justify right bottom))
   )
-  (text "TP1" (at 31.75 126.365 180)
+  (text "energize" (at 31.75 126.365 180)
     (effects (font (size 1.27 1.27)) (justify right bottom))
   )
@@
     )
   )
-  (global_label "BIT" (shape input) (at 242.57 131.445 180) (fields_autoplaced)
-    (effects (font (size 1.27 1.27)) (justify right))
-    (property "Intersheet References" "${INTERSHEET_REFS}" (id 0) (at 237.3145 131.3656 0)
-      (effects (font (size 1.27 1.27)) (justify right) hide)
-    )
-  )
   (global_label "clear" (shape input) (at 267.335 156.21 0) (fields_autoplaced)
     (effects (font (size 1.27 1.27)) (justify left))
@@
     )
   )
-  (global_label "BIT" (shape input) (at 222.885 142.24 0) (fields_autoplaced)
+  (global_label "energize" (shape input) (at 127 49.53 0) (fields_autoplaced)
     (effects (font (size 1.27 1.27)) (justify left))
-    (property "Intersheet References" "${INTERSHEET_REFS}" (id 0) (at 228.1405 142.1606 0)
-      (effects (font (size 1.27 1.27)) (justify left) hide)
-    )
-  )
-  (global_label "LBIT" (shape input) (at 266.7 133.985 0) (fields_autoplaced)
+    (property "Intersheet References" "${INTERSHEET_REFS}" (id 0) (at 137.396 49.4506 0)
+      (effects (font (size 1.27 1.27)) (justify left) hide)
+    )
+  )
+  (global_label "{slash}BIT" (shape input) (at 229.235 142.24 0) (fields_autoplaced)
     (effects (font (size 1.27 1.27)) (justify left))
-    (property "Intersheet References" "${INTERSHEET_REFS}" (id 0) (at 272.9836 133.9056 0)
+    (property "Intersheet References" "${INTERSHEET_REFS}" (id 0) (at 235.821 142.1606 0)
+      (effects (font (size 1.27 1.27)) (justify left) hide)
+    )
+  )
+  (global_label "BIT" (shape input) (at 266.7 133.985 0) (fields_autoplaced)
+    (effects (font (size 1.27 1.27)) (justify left))
+    (property "Intersheet References" "${INTERSHEET_REFS}" (id 0) (at 271.9555 133.9056 0)
       (effects (font (size 1.27 1.27)) (justify left) hide)
     )
@@
     (pin "2")
   )
-  (symbol (lib_id "Connector:TestPoint") (at 130.175 55.245 0) (unit 1)
-    (in_bom yes) (on_board yes)
-    (property "Reference" "TP1" (id 0) (at 128.27 50.165 0)
-      (effects (font (size 1.27 1.27)) (justify left))
-    )
-    (property "Value" "TestPoint" (id 1) (at 132.08 53.2129 0)
-      (effects (font (size 1.27 1.27)) (justify left) hide)
-    )
-    (property "Footprint" "" (id 2) (at 135.255 55.245 0)
-      (effects (font (size 1.27 1.27)) hide)
-    )
-    (property "Datasheet" "~" (id 3) (at 135.255 55.245 0)
-      (effects (font (size 1.27 1.27)) hide)
-    )
-    (pin "1")
-  )
   (symbol (lib_id "Device:D") (at 146.05 71.12 90) (unit 1)
     (in_bom yes) (on_board yes) (fields_autoplaced)
@@
       (reference "ROMGND") (unit 1) (value "GNDREF") (footprint "")
     )
-    (path "/6f47afab-0f52-4a8f-82f1-bde9e0c218ed"
-      (reference "TP1") (unit 1) (value "TestPoint") (footprint "")
-    )
     (path "/f38f084b-aa47-484c-af97-a87d934da924"

Commit message: still more schematic cleanup
Parts:
- gave numbers to parts that had none: 2
Other:
- note added: "4 places, decoding jad4-jad8, L12-L15"
- note added: "8 places, decoding jl, jh, jad0-jad3, L2-L9"
- note added: "measure to Vdd"
- note removed: "4 places, decoding jad4-jad8"
- note removed: "8 places, decoding jl, jh, jad0-jad3"
Changed lines of the file:
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@@
     (effects (font (size 1.27 1.27)) (justify right bottom))
   )
-  (text "8 places, decoding\njl, jh, jad0-jad3" (at 220.98 116.84 0)
+  (text "8 places, decoding\njl, jh, jad0-jad3,\nL2-L9" (at 220.98 118.745 0)
     (effects (font (size 1.27 1.27)) (justify left bottom))
   )
@@
     (effects (font (size 1.27 1.27)) (justify right bottom))
   )
+  (text "measure to Vdd" (at 57.15 125.73 0)
+    (effects (font (size 1.27 1.27)) (justify left bottom))
+  )
   (text "energize" (at 31.75 126.365 180)
     (effects (font (size 1.27 1.27)) (justify right bottom))
@@
     (effects (font (size 1.27 1.27)) (justify left bottom))
   )
-  (text "4 places, decoding\njad4-jad8 " (at 88.9 123.825 0)
+  (text "4 places, decoding\njad4-jad8, L12-L15" (at 88.9 123.825 0)
     (effects (font (size 1.27 1.27)) (justify left bottom))
   )
@@
     )
   )
-  (symbol (lib_id "Device:Q_PNP_CEB") (at 143.51 55.245 0) (mirror x) (unit 1)
+  (symbol (lib_name "Q_PNP_CEB_2") (lib_id "Device:Q_PNP_CEB") (at 143.51 55.245 0) (mirror x) (unit 1)
     (in_bom yes) (on_board yes)
     (property "Reference" "Q33" (id 0) (at 149.225 53.9749 0)
@@
   (symbol (lib_id "74xx_IEEE:74145") (at 228.6 98.425 0) (mirror y) (unit 1)
     (in_bom yes) (on_board yes) (fields_autoplaced)
-    (property "Reference" "U?" (id 0) (at 228.6 78.74 0))
+    (property "Reference" "U2" (id 0) (at 228.6 78.74 0))
     (property "Value" "74145" (id 1) (at 228.6 81.28 0))
     (property "Footprint" "" (id 2) (at 228.6 98.425 0)
@@
   (symbol (lib_id "74xx_IEEE:74145") (at 96.52 105.41 0) (unit 1)
     (in_bom yes) (on_board yes) (fields_autoplaced)
-    (property "Reference" "U?" (id 0) (at 96.52 85.725 0))
-    (property "Value" "74145" (id 1) (at 96.52 88.265 0))
+    (property "Reference" "U12" (id 0) (at 96.52 86.36 0))
+    (property "Value" "74145" (id 1) (at 96.52 88.9 0))
     (property "Footprint" "" (id 2) (at 96.52 105.41 0)
       (effects (font (size 1.27 1.27)) hide)
@@
     (pin "9")
   )
-  (symbol (lib_id "Device:Q_PNP_CEB") (at 143.51 80.01 0) (mirror x) (unit 1)
+  (symbol (lib_name "Q_PNP_CEB_1") (lib_id "Device:Q_PNP_CEB") (at 143.51 80.01 0) (mirror x) (unit 1)
     (in_bom yes) (on_board yes) (fields_autoplaced)
     (property "Reference" "Q32" (id 0) (at 148.59 78.7399 0)
@@
       (reference "TP?") (unit 1) (value "1of64") (footprint "")
     )
+    (path "/547fdf3f-1b2a-474a-abae-91623cb154ff"
+      (reference "U2") (unit 1) (value "74145") (footprint "")
+    )
     (path "/4029a5ba-5a71-478e-b921-a79251e981c4"
       (reference "U11") (unit 1) (value "7401") (footprint "")
     )
+    (path "/f6959a67-8719-49d3-9608-8ec7cdb63e2f"
+      (reference "U12") (unit 1) (value "74145") (footprint "")
+    )
     (path "/2caec8e2-d35d-4e35-973b-467fb5c8d8a5"
       (reference "U38") (unit 2) (value "74LS04") (footprint "")
     )
-    (path "/547fdf3f-1b2a-474a-abae-91623cb154ff"
-      (reference "U?") (unit 1) (value "74145") (footprint "")
-    )
     (path "/aef0b8a0-a10c-484a-bea8-74e5a02f11dd"
       (reference "U?") (unit 1) (value "74LS00") (footprint "")
     )
-    (path "/f6959a67-8719-49d3-9608-8ec7cdb63e2f"
-      (reference "U?") (unit 1) (value "74145") (footprint "")
-    )
     (path "/578792be-bc65-40ac-9353-2bbbe538bafc"
