File: wang600-docs/kicad/5969-wire-weave-rom/5969-wire-weave-rom.kicad_sch (KiCad schematic)
At the start: 38 parts, among them Q32 GT644, Q33 GT644, Q34 2N3640, U11 7426, U36 SP380A, U38 74LS04

Commit message: still more schematic cleanup
Parts:
- U38: value 74LS04 -> 7404
- gave numbers to parts that had none: 2
Other:
- note added: "(note 4) measure to Vdd"
- note added: "4 places, decoding jad4-jad8, L12-L15"
- note added: "8 places, decoding jl, jh, jad0-jad3, L2-L9"
- note removed: "(Note 4)"
- note removed: "4 places, decoding jad4-jad8"
- note removed: "8 places, decoding jl, jh, jad0-jad3"
Changed lines of the file:
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@@
     (effects (font (size 1.27 1.27)) (justify left bottom))
   )
-  (text "(Note 4)" (at 52.07 125.73 0)
+  (text "(note 4)\nmeasure to Vdd" (at 57.15 126.365 0)
     (effects (font (size 1.27 1.27)) (justify left bottom))
   )
@@
     (effects (font (size 1.27 1.27)) (justify right bottom))
   )
-  (text "8 places, decoding\njl, jh, jad0-jad3" (at 220.98 116.84 0)
+  (text "8 places, decoding\njl, jh, jad0-jad3,\nL2-L9" (at 220.98 118.745 0)
     (effects (font (size 1.27 1.27)) (justify left bottom))
   )
@@
     (effects (font (size 1.27 1.27)) (justify left bottom))
   )
-  (text "4 places, decoding\njad4-jad8 " (at 88.9 123.825 0)
+  (text "4 places, decoding\njad4-jad8, L12-L15" (at 88.9 123.825 0)
     (effects (font (size 1.27 1.27)) (justify left bottom))
   )
@@
     (pin "6")
   )
-  (symbol (lib_id "Device:Q_PNP_CEB") (at 143.51 55.245 0) (mirror x) (unit 1)
+  (symbol (lib_name "Q_PNP_CEB_2") (lib_id "Device:Q_PNP_CEB") (at 143.51 55.245 0) (mirror x) (unit 1)
     (in_bom yes) (on_board yes) (fields_autoplaced)
     (property "Reference" "Q33" (id 0) (at 149.225 53.9749 0)
@@
     (in_bom yes) (on_board yes)
     (property "Reference" "U38" (id 0) (at 259.08 157.48 0))
-    (property "Value" "74LS04" (id 1) (at 257.81 150.495 0)
-      (effects (font (size 1.27 1.27)) hide)
-    )
+    (property "Value" "7404" (id 1) (at 255.905 153.67 0))
     (property "Footprint" "" (id 2) (at 257.81 157.48 0)
       (effects (font (size 1.27 1.27)) hide)
@@
   (symbol (lib_id "74xx:74LS26") (at 39.37 46.99 0) (unit 1)
     (in_bom yes) (on_board yes)
-    (property "Reference" "U11" (id 0) (at 39.37 41.91 0))
-    (property "Value" "7426" (id 1) (at 39.37 46.99 0))
+    (property "Reference" "U11" (id 0) (at 39.37 46.99 0))
+    (property "Value" "7426" (id 1) (at 41.91 41.91 0))
     (property "Footprint" "" (id 2) (at 39.37 46.99 0)
       (effects (font (size 1.27 1.27)) hide)
@@
   (symbol (lib_id "74xx_IEEE:74145") (at 228.6 98.425 0) (mirror y) (unit 1)
     (in_bom yes) (on_board yes) (fields_autoplaced)
-    (property "Reference" "U?" (id 0) (at 228.6 78.74 0))
+    (property "Reference" "U2" (id 0) (at 228.6 78.74 0))
     (property "Value" "74145" (id 1) (at 228.6 81.28 0))
     (property "Footprint" "" (id 2) (at 228.6 98.425 0)
@@
     (in_bom yes) (on_board yes)
     (property "Reference" "U38" (id 0) (at 156.845 157.48 0))
-    (property "Value" "74LS04" (id 1) (at 158.115 150.495 0)
-      (effects (font (size 1.27 1.27)) hide)
-    )
+    (property "Value" "7404" (id 1) (at 159.385 153.67 0))
     (property "Footprint" "" (id 2) (at 158.115 157.48 0)
       (effects (font (size 1.27 1.27)) hide)
@@
     (pin "2")
   )
-  (symbol (lib_id "Device:Q_PNP_CEB") (at 75.565 46.99 0) (mirror x) (unit 1)
+  (symbol (lib_name "Q_PNP_CEB_1") (lib_id "Device:Q_PNP_CEB") (at 75.565 46.99 0) (mirror x) (unit 1)
     (in_bom yes) (on_board yes)
     (property "Reference" "Q34" (id 0) (at 73.025 42.545 0)
@@
   (symbol (lib_id "74xx_IEEE:74145") (at 96.52 105.41 0) (unit 1)
     (in_bom yes) (on_board yes) (fields_autoplaced)
-    (property "Reference" "U?" (id 0) (at 96.52 85.725 0))
-    (property "Value" "74145" (id 1) (at 96.52 88.265 0))
+    (property "Reference" "U12" (id 0) (at 96.52 86.36 0))
+    (property "Value" "74145" (id 1) (at 96.52 88.9 0))
     (property "Footprint" "" (id 2) (at 96.52 105.41 0)
       (effects (font (size 1.27 1.27)) hide)
@@
       (reference "TP?") (unit 1) (value "1of64") (footprint "")
     )
+    (path "/547fdf3f-1b2a-474a-abae-91623cb154ff"
+      (reference "U2") (unit 1) (value "74145") (footprint "")
+    )
     (path "/4029a5ba-5a71-478e-b921-a79251e981c4"
       (reference "U11") (unit 1) (value "7426") (footprint "")
     )
+    (path "/f6959a67-8719-49d3-9608-8ec7cdb63e2f"
+      (reference "U12") (unit 1) (value "74145") (footprint "")
+    )
     (path "/4ee56eaa-82d2-40a0-8d6c-b649233d6ceb"
       (reference "U36") (unit 1) (value "SP380A") (footprint "")
@@
     )
     (path "/7749d8be-dd68-427a-aeec-b971b41fb048"
-      (reference "U38") (unit 1) (value "74LS04") (footprint "")
+      (reference "U38") (unit 1) (value "7404") (footprint "")
     )
     (path "/2caec8e2-d35d-4e35-973b-467fb5c8d8a5"
-      (reference "U38") (unit 2) (value "74LS04") (footprint "")
-    )
-    (path "/547fdf3f-1b2a-474a-abae-91623cb154ff"
-      (reference "U?") (unit 1) (value "74145") (footprint "")
-    )
-    (path "/f6959a67-8719-49d3-9608-8ec7cdb63e2f"
-      (reference "U?") (unit 1) (value "74145") (footprint "")
-    )
-  )
+      (reference "U38") (unit 2) (value "7404") (footprint "")
+    )
+  )
