File: wang600-docs/kicad/6184-etc-KA-KB-handling/6184-etc-KA-KB-handling.kicad_sch (KiCad schematic)
At the start: 34 parts, among them Q1 Q_NPN_BCE, Q2 Q_NPN_BCE, Q3 Q_NPN_BCE, Q4 Q_NPN_BCE

Commit message: w600: fixup details
Connections:
- net GND: now also C6.1; no longer C6.2
- net at D6.1 (K), Q4.3 (E), R16.2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: now also C6.2; no longer C6.1
Other:
- note added: "-1.4V"
- note added: "OR (w/delay)"
- note added: "pre-Z2 Z2 LOCK 1 -1.4V (KBL) 0 4.2V? 1"
- note removed: "NOR (w/delay)"
- moved on the sheet: C6, D5, D6, R16, R17
